Commit message: update urdf

File: wsg50_description/urdf/wsg50.urdf.xacro (robot description, xacro)
@@ -1,11 +1,11 @@
 <?xml version="1.0"?>
 <robot xmlns:xacro="http://www.ros.org/wiki/xacro">
-    <xacro:macro name="wsg50" params="prefix finger_length finger_tip *origin">
+    <xacro:macro name="wsg50" params="prefix parent finger_length finger_tip *origin">
         <joint name="${prefix}_gripper_joint" type="fixed">
-            <insert_block name="origin"/>
+            <xacro:insert_block name="origin" />
             <parent link="${parent}"/>
-            <child link="${name}_base_link"/>
+            <child link="${prefix}_base_link"/>
         </joint>
-         <link name="${name}_base_link">
+         <link name="${prefix}_base_link">
             <inertial>
                 <mass value="0.25" />
@@ -29,4 +29,92 @@
             </collision>
         </link>
+        <gazebo reference="${prefix}_base_link">
+            <material>Gazebo/Grey</material>
+            <turnGravityOff>false</turnGravityOff>
+        </gazebo>
+        <joint name="${prefix}_center_joint" type="fixed">
+            <origin xyz="0 0 ${finger_length}" rpy="0 0 0" />      <!--origin xyz="-0.0067 0 0.049" rpy="0 0 0" /-->
+            <parent link="${prefix}_base_link"/>
+            <child link="${prefix}_center" />
+        </joint>
+        <link name="${prefix}_center" />
+        <!-- GRIPPER LEFT -->
+        <link name="${prefix}_gripper_left">
+            <inertial>
+                <mass value="0.1" />
+                <origin xyz="0 0 0" />
+                <inertia ixx="1.0" ixy="0.0" ixz="0.0"
+                    iyy="1.0" iyz="0.0"
+                    izz="1.0" />
+            </inertial>
+            <visual>
+                <origin xyz="0.0 0 0" rpy="0 0 0" />
+                <geometry>
+                    <mesh filename="package://wsg50_description/meshes/WSG_FMF.dae" scale="0.001 0.001 0.001"/>
+                </geometry>
+                <material name="black">
+                    <color rgba="0 0 0 0"/>
+                </material>
+            </visual>
+            <collision>
+                <origin xyz="0 0 0" rpy="0 0 0" />
+                <geometry>
+                    <mesh filename="package://wsg50_description/meshes/WSG_FMF.stl" scale="0.001 0.001 0.001"/>
+                </geometry>
+            </collision>
+            <contact_coefficients kd="1.0" kp="1000.0" mu="0"/>
+        </link>
+        <gazebo reference="${prefix}_gripper_left">
+            <material>Gazebo/Blue</material>
+            <turnGravityOff>false</turnGravityOff>
+        </gazebo>
+        <joint name="${prefix}_finger_left_joint" type="fixed">
+            <limit lower="-0.055" upper="-0.0027" effort="1.0" velocity="1.0"/>
+            <origin xyz="0 0 0.3" rpy="0 0 0" />      <!--origin xyz="-0.0067 0 0.049" rpy="0 0 0" /-->
+            <parent link="${prefix}_base_link"/>
+            <child link="${prefix}_gripper_left" />
+            <dynamics friction="100" damping="100" />
+            <axis xyz="1 0 0"/>
+            <limit effort="100" velocity="100"/>
+        </joint>
+         <!-- GRIPPER RIGHT -->
+        <link name="${prefix}_gripper_right">
+            <inertial>
+                <mass value="0.1" />
+                <origin xyz="0 0 0" />
+            <inertia ixx="1.0" ixy="0.0" ixz="0.0"
+                    iyy="1.0" iyz="0.0"
+                    izz="1.0" />
+            </inertial>
+            <visual>
+                <origin xyz="0.0 0 0" rpy="0 0 0" />
+                <geometry>
+                    <mesh filename="package://wsg50_description/meshes/WSG_FMF.dae" scale="1 1 1"/>
+                </geometry>
+                <material name="black">
+                    <color rgba="0 0 0 0"/>
+                </material>
+            </visual>
+            <collision>
+                <origin xyz="0 0 0" rpy="0 0 0" />
+                <geometry>
+                    <mesh filename="package://wsg50_description/meshes/WSG_FMF.stl" scale="0.001 0.001 0.001"/>
+                </geometry>
+            </collision>
+            <contact_coefficients kd="1.0" kp="1000.0" mu="0"/>
+        </link>
+        <gazebo reference="gripper_right">
+            <material>Gazebo/White</material>
+            <turnGravityOff>false</turnGravityOff>
+        </gazebo>
+        <joint name="${prefix}_finger_right_joint" type="fixed">
+            <limit lower="0.0027" upper="0.055" effort="1.0" velocity="1.0"/>
+            <origin xyz="0 0 0.3" rpy="0 0 3.14159" />
+            <parent link="${prefix}_base_link"/>
+            <child link="${prefix}_gripper_right" />
+            <axis xyz="-1 0 0"/>
+            <dynamics friction="100" damping="100" />
+            <limit effort="100" velocity="100"/>
+        </joint>
     </xacro:macro>
 </robot>

Commit message: update urdf

File: wsg50_description/urdf/wsg50.urdf.xacro (robot description, xacro)
@@ -51,5 +51,5 @@
                 <origin xyz="0.0 0 0" rpy="0 0 0" />
                 <geometry>
-                    <mesh filename="package://wsg50_description/meshes/WSG_FMF.dae" scale="0.001 0.001 0.001"/>
+                    <mesh filename="package://wsg50_description/meshes/WSG_FMF.dae" />
                 </geometry>
                 <material name="black">
@@ -60,5 +60,5 @@
                 <origin xyz="0 0 0" rpy="0 0 0" />
                 <geometry>
-                    <mesh filename="package://wsg50_description/meshes/WSG_FMF.stl" scale="0.001 0.001 0.001"/>
+                    <mesh filename="package://wsg50_description/meshes/WSG_FMF.stl" />
                 </geometry>
             </collision>
@@ -71,5 +71,5 @@
         <joint name="${prefix}_finger_left_joint" type="fixed">
             <limit lower="-0.055" upper="-0.0027" effort="1.0" velocity="1.0"/>
-            <origin xyz="0 0 0.3" rpy="0 0 0" />      <!--origin xyz="-0.0067 0 0.049" rpy="0 0 0" /-->
+            <origin xyz="0 0 0.09" rpy="0 0 0" />      <!--origin xyz="-0.0067 0 0.049" rpy="0 0 0" /-->
             <parent link="${prefix}_base_link"/>
             <child link="${prefix}_gripper_left" />
@@ -90,5 +90,5 @@
                 <origin xyz="0.0 0 0" rpy="0 0 0" />
                 <geometry>
-                    <mesh filename="package://wsg50_description/meshes/WSG_FMF.dae" scale="1 1 1"/>
+                    <mesh filename="package://wsg50_description/meshes/WSG_FMF.dae" />
                 </geometry>
                 <material name="black">
@@ -99,5 +99,5 @@
                 <origin xyz="0 0 0" rpy="0 0 0" />
                 <geometry>
-                    <mesh filename="package://wsg50_description/meshes/WSG_FMF.stl" scale="0.001 0.001 0.001"/>
+                    <mesh filename="package://wsg50_description/meshes/WSG_FMF.stl"/>
                 </geometry>
             </collision>
@@ -110,5 +110,5 @@
         <joint name="${prefix}_finger_right_joint" type="fixed">
             <limit lower="0.0027" upper="0.055" effort="1.0" velocity="1.0"/>
-            <origin xyz="0 0 0.3" rpy="0 0 3.14159" />
+            <origin xyz="0 0 0.09" rpy="0 0 3.14159" />
             <parent link="${prefix}_base_link"/>
             <child link="${prefix}_gripper_right" />

Commit message: update gripper fingures

File: wsg50_description/urdf/wsg50.urdf.xacro (robot description, xacro)
@@ -49,16 +49,14 @@
             </inertial>
             <visual>
-                <origin xyz="0.0 0 0" rpy="0 0 0" />
+                <origin xyz="0 0 0" rpy="0 0 0" />
+                <material name="grey" />
                 <geometry>
-                    <mesh filename="package://wsg50_description/meshes/WSG_FMF.dae" />
+                    <mesh filename="package://wsg50_description/meshes/kuka_gripper_2.dae" />
                 </geometry>
-                <material name="black">
-                    <color rgba="0 0 0 0"/>
-                </material>
             </visual>
             <collision>
                 <origin xyz="0 0 0" rpy="0 0 0" />
                 <geometry>
-                    <mesh filename="package://wsg50_description/meshes/WSG_FMF.stl" />
+                    <mesh filename="package://wsg50_description/meshes/kuka_gripper_2.stl" />
                 </geometry>
             </collision>
@@ -71,5 +69,5 @@
         <joint name="${prefix}_finger_left_joint" type="fixed">
             <limit lower="-0.055" upper="-0.0027" effort="1.0" velocity="1.0"/>
-            <origin xyz="0 0 0.09" rpy="0 0 0" />      <!--origin xyz="-0.0067 0 0.049" rpy="0 0 0" /-->
+            <origin xyz="0.08 0 0.16" rpy="3.1457 0 3.1457" />      <!--origin xyz="-0.0067 0 0.049" rpy="0 0 0" /-->
             <parent link="${prefix}_base_link"/>
             <child link="${prefix}_gripper_left" />
@@ -89,15 +87,13 @@
             <visual>
                 <origin xyz="0.0 0 0" rpy="0 0 0" />
+                <material name="grey" />
                 <geometry>
-                    <mesh filename="package://wsg50_description/meshes/WSG_FMF.dae" />
+                    <mesh filename="package://wsg50_description/meshes/kuka_gripper_2.dae" />
                 </geometry>
-                <material name="black">
-                    <color rgba="0 0 0 0"/>
-                </material>
             </visual>
             <collision>
                 <origin xyz="0 0 0" rpy="0 0 0" />
                 <geometry>
-                    <mesh filename="package://wsg50_description/meshes/WSG_FMF.stl"/>
+                    <mesh filename="package://wsg50_description/meshes/kuka_gripper_2.stl"/>
                 </geometry>
             </collision>
@@ -110,5 +106,5 @@
         <joint name="${prefix}_finger_right_joint" type="fixed">
             <limit lower="0.0027" upper="0.055" effort="1.0" velocity="1.0"/>
-            <origin xyz="0 0 0.09" rpy="0 0 3.14159" />
+            <origin xyz="-0.08 0 0.16" rpy="3.14159 0 0" />
             <parent link="${prefix}_base_link"/>
             <child link="${prefix}_gripper_right" />
@@ -117,4 +113,26 @@
             <limit effort="100" velocity="100"/>
         </joint>
+        <!-- <link name="object">
+            <inertial>
+                <mass value="100"/>
+                <origin xyz="0 0 0" />
+                <inertia  ixx="1" ixy="0.0"  ixz="0.0"  iyy="1"  iyz="0.0"  izz="1" />
+            </inertial>
+            <visual>
+                <origin rpy="0 0 0" xyz="0 0 0"/>
+                <geometry>
+                    <box size="0.08 0.08 0.4"/>
+                </geometry>
+                <material name="white">
+                    <color rgba="1.0 1.0 1.0 1.0"/>
+                </material>
+            </visual>
+            <collision>
+                <origin rpy="0 0 0" xyz="0 0 0"/>
+                <geometry>
+                    <box size="0.08 0.08 0.4"/>
+                </geometry>
+            </collision>
+        </link> -->
     </xacro:macro>
 </robot>

Commit message: update model for collision factors

File: wsg50_description/urdf/wsg50.urdf.xacro (robot description, xacro)
@@ -16,5 +16,6 @@
                 <origin xyz="0.0 0 0" rpy="0 0 0" />
                 <geometry>
-                    <mesh filename="package://wsg50_description/meshes/WSG50_110.stl" scale="1 1 1"/>
+                    <box size="0.20 0.09 0.0735"/>
+                    <!-- <mesh filename="package://wsg50_description/meshes/WSG50_110.stl" scale="1 1 1"/> -->
                 </geometry>
                 <material name="grey">
@@ -25,5 +26,6 @@
                 <origin xyz="0.0 0 0" rpy="0 0 0" />
                 <geometry>
-                    <mesh filename="package://wsg50_description/meshes/WSG50_110.stl" scale="1 1 1"/>
+                    <box size="0.25 0.09 0.0735"/>
+                    <!-- <mesh filename="package://wsg50_description/meshes/WSG50_110.stl" scale="1 1 1"/> -->
                 </geometry>
             </collision>
@@ -69,5 +71,5 @@
         <joint name="${prefix}_finger_left_joint" type="fixed">
             <limit lower="-0.055" upper="-0.0027" effort="1.0" velocity="1.0"/>
-            <origin xyz="0.08 0 0.16" rpy="3.1457 0 3.1457" />      <!--origin xyz="-0.0067 0 0.049" rpy="0 0 0" /-->
+            <origin xyz="0.08 0 0.12" rpy="3.1457 0 3.1457" />      <!--origin xyz="-0.0067 0 0.049" rpy="0 0 0" /-->
             <parent link="${prefix}_base_link"/>
             <child link="${prefix}_gripper_left" />
@@ -106,5 +108,5 @@
         <joint name="${prefix}_finger_right_joint" type="fixed">
             <limit lower="0.0027" upper="0.055" effort="1.0" velocity="1.0"/>
-            <origin xyz="-0.08 0 0.16" rpy="3.14159 0 0" />
+            <origin xyz="-0.08 0 0.12" rpy="3.14159 0 0" />
             <parent link="${prefix}_base_link"/>
             <child link="${prefix}_gripper_right" />
